File: PCB/RecyclingPad_embedded/RecyclingPad_embedded.kicad_pcb (KiCad board)
At the start: 2 copper layers, 80.5 x 80.5 mm, 40 parts, among them U1 ATmega32U2-AU, U2 SRV05-4, X1 Crystal_GND24_Small

Commit message: Embedded version of the RecyclingPad
Parts:
- D1, D2, D3, D4, D5, D6, D7, D8, D9: footprint Diode_SMD:D_SOD-123 -> Diode_SMD:D_SOD-323F
Routing:
- net ROW0: track 61.9 -> 63.6 mm
- net ROW1: track 82.0 -> 83.7 mm
- net ROW2: track 103.4 -> 104.9 mm
- net Net-(D7-Pad2): track 7.95 -> 8.56 mm
- net Net-(D4-Pad2): track 7.95 -> 8.55 mm
- net Net-(D9-Pad2): track 7.95 -> 8.50 mm
- net Net-(D8-Pad2): track 7.95 -> 8.50 mm
- net Net-(D6-Pad2): track 7.95 -> 8.50 mm
- net Net-(D5-Pad2): track 7.95 -> 8.50 mm
- net Net-(D3-Pad2): track 7.95 -> 8.50 mm
- net Net-(D1-Pad2): track 7.95 -> 8.50 mm
- net GND: track 10.9 -> 10.4 mm
