File: PCB/RecyclingPad_embedded/RecyclingPad_embedded.kicad_sch (KiCad schematic)
At the start: 36 parts, among them U1 ATmega32U2-AU, U2 SRV05-4, X1 Crystal_GND24_Small

Commit message: Embedded version of the RecyclingPad
Parts:
- C1: LCSC C91245 -> (none); LCSC Part (none) -> C91245
- C2, C3: LCSC C1804 -> (none); LCSC Part (none) -> C1804
- C4, C5: LCSC C49678 -> (none); LCSC Part (none) -> C49678
- C6: LCSC C28323 -> (none); LCSC Part (none) -> C28323
- D1, D2, D3, D4, D5, D6, D7, D8, D9: footprint Diode_SMD:D_SOD-123 -> Diode_SMD:D_SOD-323; symbol Diode:1N4148W -> Diode:1N4148WS; LCSC Part (none) -> C2128
- F1: LCSC C69688 -> (none); LCSC Part (none) -> C69688
- R1, R2: LCSC C17561 -> (none); LCSC Part (none) -> C17561
- R3, R7: LCSC C17414 -> (none); LCSC Part (none) -> C17414
- R4, R5: LCSC C27834 -> (none); LCSC Part (none) -> C27834
- RESET1: LCSC C318884 -> (none); LCSC Part (none) -> C318884
- U1: LCSC C618733 -> (none); LCSC Part (none) -> C618733
- U2: LCSC C85364 -> (none); LCSC Part (none) -> C85364
- USB1: LCSC C165948 -> (none); LCSC Part (none) -> C165948
- X1: LCSC C13738 -> (none); LCSC Part (none) -> C13738
