File: PCB/RecyclingPad/RecyclingPad.kicad_sch (KiCad schematic)
At the start: 20 parts

Commit message: Update recyclingPad v1.0
Connections:
- net ROW0: now also B1.13 (*10), D4.C, D5.C, D6.C; no longer B1.15 (12(MISO)), D1.C, D2.C, D3.C
- net ROW1: now also B1.15 (12(MISO)), D1.C, D2.C, D3.C; no longer B1.13 (*10), D4.C, D5.C, D6.C
Changed lines of the file:
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@@
   (title_block
     (title "RecyclingPad")
-    (date "2022-06-22")
-    (rev "0.1x")
+    (date "2022-07-06")
+    (rev "1.0x")
     (company "deveth0")
   )
@@
     (effects (font (size 1.2446 1.2446)) (justify left bottom))
   )
-  (label "ROW1" (at 91.44 90.17 0)
+  (label "ROW0" (at 91.44 90.17 0)
     (effects (font (size 1.2446 1.2446)) (justify left bottom))
   )
@@
     (effects (font (size 1.2446 1.2446)) (justify left bottom))
   )
-  (label "ROW1" (at 264.16 127 0)
+  (label "ROW0" (at 264.16 127 0)
     (effects (font (size 1.27 1.27)) (justify left bottom))
   )
@@
     (effects (font (size 1.2446 1.2446)) (justify left bottom))
   )
-  (label "ROW0" (at 30.48 90.17 0)
-    (effects (font (size 1.2446 1.2446)) (justify left bottom))
-  )
-  (label "ROW0" (at 264.16 121.92 0)
+  (label "ROW1" (at 30.48 90.17 0)
+    (effects (font (size 1.2446 1.2446)) (justify left bottom))
+  )
+  (label "ROW1" (at 264.16 121.92 0)
     (effects (font (size 1.2446 1.2446)) (justify left bottom))
   )
@@
   (symbol (lib_id "dumbpad-eagle-import:GND") (at 59.69 63.5 0) (unit 1)
     (in_bom yes) (on_board yes)
-    (property "Reference" "#GND?" (id 0) (at 59.69 63.5 0)
+    (property "Reference" "#GND0104" (id 0) (at 59.69 63.5 0)
       (effects (font (size 1.27 1.27)) hide)
     )
@@
     )
     (path "/48c7fbc2-41c9-4c8f-885b-69a9fd2e1c25"
-      (reference "#GND?") (unit 1) (value "GND") (footprint "")
+      (reference "#GND0104") (unit 1) (value "GND") (footprint "")
     )
     (path "/d74fd4e6-dda5-4b0a-9281-50912d229d8f"
